File: nighthawk.kicad_sch (KiCad schematic)
At the start: 58 parts, among them M1 BURRO, Q1 2N7000, Q2 NPN, SW1 SW_Push_Open, SW2 SW_Push, SW3 SW_Push, SW4 SW_SPST, SW5 SW_Push, SW6 SW_Push, SW7 SW_Push

Commit message: rev 3
Parts:
- removed R4: 1k, symbol Device:R
- added F5: 2A, symbol Device:Fuse
Connections:
- net KEY_NO_2: now also F5.2
- net BOBINA renamed BOBINAS
- new net RELAY+: F5.1
- no-connect marks 11 -> 12
Other:
- moved on the sheet: F4, L1, L2
